File: PCD_PLV005_Beyla/AvionicsHeartbeat.sch (KiCad schematic (older format))
At the start: 30 parts, among them Q1 DMG2302UK-7, Q2 DMP2123L-7, U2 74HC266, U3 74HC08, U4 74HC21, U5 74LVC1G17, U6 LTC6993xS6-1

Commit message: Beyla Initial Layout
Co-Authored-By: cronin11 <74317819+cronin11@users.noreply.github.com>
Parts:
- C2, C3, C4, C5, C6: footprint Capacitor_SMD:C_0603_1608Metric_Pad1.05x0.95mm_HandSolder -> Capacitor_SMD:C_0603_1608Metric_Pad1.08x0.95mm_HandSolder
- C7: footprint (none) -> Capacitor_SMD:C_0603_1608Metric_Pad1.08x0.95mm_HandSolder
- R1, R10, R11, R12, R14, R16, R17, R2, R3, R4, R5, R6, R7, R8, R9: footprint (none) -> Resistor_SMD:R_0603_1608Metric_Pad0.98x0.95mm_HandSolder
Changed lines of the file:
@@
 EESchema Schematic File Version 4
-LIBS:PCB_PLV005_Beyla-cache
-EELAYER 29 0
+EELAYER 30 0
 EELAYER END
 $Descr A4 11693 8268
@@
 F 0 "R1" V 1805 5050 50  0000 C CNN
 F 1 "0" V 1714 5050 50  0000 C CNN
-F 2 "" V 1640 5040 50  0001 C CNN
+F 2 "Resistor_SMD:R_0603_1608Metric_Pad0.98x0.95mm_HandSolder" V 1640 5040 50  0001 C CNN
 F 3 "~" H 1600 5050 50  0001 C CNN
 	1    1600 5050
@@
 F 0 "R2" V 1805 5600 50  0000 C CNN
 F 1 "0" V 1714 5600 50  0000 C CNN
-F 2 "" V 1640 5590 50  0001 C CNN
+F 2 "Resistor_SMD:R_0603_1608Metric_Pad0.98x0.95mm_HandSolder" V 1640 5590 50  0001 C CNN
 F 3 "~" H 1600 5600 50  0001 C CNN
 	1    1600 5600
@@
 F 0 "R3" V 1805 6150 50  0000 C CNN
 F 1 "0" V 1714 6150 50  0000 C CNN
-F 2 "" V 1640 6140 50  0001 C CNN
+F 2 "Resistor_SMD:R_0603_1608Metric_Pad0.98x0.95mm_HandSolder" V 1640 6140 50  0001 C CNN
 F 3 "~" H 1600 6150 50  0001 C CNN
 	1    1600 6150
@@
 F 0 "R4" V 1805 6700 50  0000 C CNN
 F 1 "0" V 1714 6700 50  0000 C CNN
-F 2 "" V 1640 6690 50  0001 C CNN
+F 2 "Resistor_SMD:R_0603_1608Metric_Pad0.98x0.95mm_HandSolder" V 1640 6690 50  0001 C CNN
 F 3 "~" H 1600 6700 50  0001 C CNN
 	1    1600 6700
@@
 F 0 "R5" H 1868 4896 50  0000 L CNN
 F 1 "DNP" H 1868 4805 50  0000 L CNN
-F 2 "" V 1840 4840 50  0001 C CNN
+F 2 "Resistor_SMD:R_0603_1608Metric_Pad0.98x0.95mm_HandSolder" V 1840 4840 50  0001 C CNN
 F 3 "~" H 1800 4850 50  0001 C CNN
 	1    1800 4850
@@
 F 0 "R6" H 1868 5446 50  0000 L CNN
 F 1 "DNP" H 1868 5355 50  0000 L CNN
-F 2 "" V 1840 5390 50  0001 C CNN
+F 2 "Resistor_SMD:R_0603_1608Metric_Pad0.98x0.95mm_HandSolder" V 1840 5390 50  0001 C CNN
 F 3 "~" H 1800 5400 50  0001 C CNN
 	1    1800 5400
@@
 F 0 "R7" H 1868 5996 50  0000 L CNN
 F 1 "DNP" H 1868 5905 50  0000 L CNN
-F 2 "" V 1840 5940 50  0001 C CNN
+F 2 "Resistor_SMD:R_0603_1608Metric_Pad0.98x0.95mm_HandSolder" V 1840 5940 50  0001 C CNN
 F 3 "~" H 1800 5950 50  0001 C CNN
 	1    1800 5950
@@
 F 0 "R8" H 1868 6546 50  0000 L CNN
 F 1 "DNP" H 1868 6455 50  0000 L CNN
-F 2 "" V 1840 6490 50  0001 C CNN
+F 2 "Resistor_SMD:R_0603_1608Metric_Pad0.98x0.95mm_HandSolder" V 1840 6490 50  0001 C CNN
 F 3 "~" H 1800 6500 50  0001 C CNN
 	1    1800 6500
@@
 F 0 "R11" H 5718 3696 50  0000 L CNN
 F 1 "604K" H 5718 3605 50  0000 L CNN
-F 2 "" V 5690 3640 50  0001 C CNN
+F 2 "Resistor_SMD:R_0603_1608Metric_Pad0.98x0.95mm_HandSolder" V 5690 3640 50  0001 C CNN
 F 3 "~" H 5650 3650 50  0001 C CNN
 	1    5650 3650
@@
 F 0 "R9" H 5418 3096 50  0000 L CNN
 F 1 "1M" H 5418 3005 50  0000 L CNN
-F 2 "" V 5390 3040 50  0001 C CNN
+F 2 "Resistor_SMD:R_0603_1608Metric_Pad0.98x0.95mm_HandSolder" V 5390 3040 50  0001 C CNN
 F 3 "~" H 5350 3050 50  0001 C CNN
 	1    5350 3050
@@
 F 0 "R10" H 5418 3696 50  0000 L CNN
 F 1 "280K" H 5418 3605 50  0000 L CNN
-F 2 "" V 5390 3640 50  0001 C CNN
+F 2 "Resistor_SMD:R_0603_1608Metric_Pad0.98x0.95mm_HandSolder" V 5390 3640 50  0001 C CNN
 F 3 "~" H 5350 3650 50  0001 C CNN
 	1    5350 3650
@@
 F 0 "R14" H 7618 3596 50  0000 L CNN
 F 1 "47K" H 7618 3505 50  0000 L CNN
-F 2 "" V 7590 3540 50  0001 C CNN
+F 2 "Resistor_SMD:R_0603_1608Metric_Pad0.98x0.95mm_HandSolder" V 7590 3540 50  0001 C CNN
 F 3 "~" H 7550 3550 50  0001 C CNN
 	1    7550 3550
@@
 F 0 "R12" H 6968 2946 50  0000 L CNN
 F 1 "47K" H 6968 2855 50  0000 L CNN
-F 2 "" V 6940 2890 50  0001 C CNN
+F 2 "Resistor_SMD:R_0603_1608Metric_Pad0.98x0.95mm_HandSolder" V 6940 2890 50  0001 C CNN
 F 3 "~" H 6900 2900 50  0001 C CNN
 	1    6900 2900
@@
 F 0 "C7" H 7565 1446 50  0000 L CNN
 F 1 "1uF" H 7565 1355 50  0000 L CNN
-F 2 "" H 7488 1250 50  0001 C CNN
+F 2 "Capacitor_SMD:C_0603_1608Metric_Pad1.08x0.95mm_HandSolder" H 7488 1250 50  0001 C CNN
 F 3 "~" H 7450 1400 50  0001 C CNN
 	1    7450 1400
@@
 F 0 "R16" H 4318 3846 50  0000 L CNN
 F 1 "1K" H 4318 3755 50  0000 L CNN
-F 2 "" V 4290 3790 50  0001 C CNN
+F 2 "Resistor_SMD:R_0603_1608Metric_Pad0.98x0.95mm_HandSolder" V 4290 3790 50  0001 C CNN
 F 3 "~" H 4250 3800 50  0001 C CNN
 	1    4250 3800
@@
 F 0 "R17" H 8918 3896 50  0000 L CNN
 F 1 "1K" H 8918 3805 50  0000 L CNN
-F 2 "" V 8890 3840 50  0001 C CNN
+F 2 "Resistor_SMD:R_0603_1608Metric_Pad0.98x0.95mm_HandSolder" V 8890 3840 50  0001 C CNN
 F 3 "~" H 8850 3850 50  0001 C CNN
 	1    8850 3850
@@
 F 0 "C2" H 5315 1446 50  0000 L CNN
 F 1 "0.1uF" H 5315 1355 50  0000 L CNN
-F 2 "Capacitor_SMD:C_0603_1608Metric_Pad1.05x0.95mm_HandSolder" H 5238 1250 50  0001 C CNN
+F 2 "Capacitor_SMD:C_0603_1608Metric_Pad1.08x0.95mm_HandSolder" H 5238 1250 50  0001 C CNN
 F 3 "https://www.yageo.com/upload/media/product/productsearch/datasheet/mlcc/UPY-GPHC_X7R_6.3V-to-50V_18.pdf" H 5200 1400 50  0001 C CNN
 F 4 "311-1341-1-ND" H 5200 1400 50  0001 C CNN "Digikey"
@@
 F 0 "C3" H 5765 1446 50  0000 L CNN
 F 1 "0.1uF" H 5765 1355 50  0000 L CNN
-F 2 "Capacitor_SMD:C_0603_1608Metric_Pad1.05x0.95mm_HandSolder" H 5688 1250 50  0001 C CNN
+F 2 "Capacitor_SMD:C_0603_1608Metric_Pad1.08x0.95mm_HandSolder" H 5688 1250 50  0001 C CNN
 F 3 "https://www.yageo.com/upload/media/product/productsearch/datasheet/mlcc/UPY-GPHC_X7R_6.3V-to-50V_18.pdf" H 5650 1400 50  0001 C CNN
 F 4 "311-1341-1-ND" H 5650 1400 50  0001 C CNN "Digikey"
@@
 F 0 "C4" H 6215 1446 50  0000 L CNN
 F 1 "0.1uF" H 6215 1355 50  0000 L CNN
-F 2 "Capacitor_SMD:C_0603_1608Metric_Pad1.05x0.95mm_HandSolder" H 6138 1250 50  0001 C CNN
+F 2 "Capacitor_SMD:C_0603_1608Metric_Pad1.08x0.95mm_HandSolder" H 6138 1250 50  0001 C CNN
 F 3 "https://www.yageo.com/upload/media/product/productsearch/datasheet/mlcc/UPY-GPHC_X7R_6.3V-to-50V_18.pdf" H 6100 1400 50  0001 C CNN
 F 4 "311-1341-1-ND" H 6100 1400 50  0001 C CNN "Digikey"
@@
 F 0 "C5" H 6665 1446 50  0000 L CNN
 F 1 "0.1uF" H 6665 1355 50  0000 L CNN
-F 2 "Capacitor_SMD:C_0603_1608Metric_Pad1.05x0.95mm_HandSolder" H 6588 1250 50  0001 C CNN
+F 2 "Capacitor_SMD:C_0603_1608Metric_Pad1.08x0.95mm_HandSolder" H 6588 1250 50  0001 C CNN
 F 3 "https://www.yageo.com/upload/media/product/productsearch/datasheet/mlcc/UPY-GPHC_X7R_6.3V-to-50V_18.pdf" H 6550 1400 50  0001 C CNN
 F 4 "311-1341-1-ND" H 6550 1400 50  0001 C CNN "Digikey"
@@
 F 0 "C6" H 7115 1446 50  0000 L CNN
 F 1 "0.1uF" H 7115 1355 50  0000 L CNN
-F 2 "Capacitor_SMD:C_0603_1608Metric_Pad1.05x0.95mm_HandSolder" H 7038 1250 50  0001 C CNN
+F 2 "Capacitor_SMD:C_0603_1608Metric_Pad1.08x0.95mm_HandSolder" H 7038 1250 50  0001 C CNN
 F 3 "https://www.yageo.com/upload/media/product/productsearch/datasheet/mlcc/UPY-GPHC_X7R_6.3V-to-50V_18.pdf" H 7000 1400 50  0001 C CNN
 F 4 "311-1341-1-ND" H 7000 1400 50  0001 C CNN "Digikey"
