File: PCD_PLV005_Beyla/PCB_PLV005_Beyla.sch (KiCad schematic (older format))
At the start: 8 parts, among them J1 PWR/QB, J2 Switch_In

Commit message: Beyla Layout Fixes, Initial Routing
Parts:
- J1: footprint Connector_Molex:Molex_Micro-Fit_3.0_43045-1200_2x06_P3.00mm_Horizontal -> Connector_Molex:Molex_Micro-Fit_3.0_43045-0800_2x04_P3.00mm_Horizontal
Changed lines of the file:
@@
 F 0 "J1" H 7380 4242 50  0000 L CNN
 F 1 "PWR/QB" H 7380 4151 50  0000 L CNN
-F 2 "Connector_Molex:Molex_Micro-Fit_3.0_43045-1200_2x06_P3.00mm_Horizontal" H 7300 4250 50  0001 C CNN
+F 2 "Connector_Molex:Molex_Micro-Fit_3.0_43045-0800_2x04_P3.00mm_Horizontal" H 7300 4250 50  0001 C CNN
 F 3 "https://www.molex.com/pdm_docs/ps/PS-43045.pdf" H 7300 4250 50  0001 C CNN
 	1    7300 4250
