File: PCB_PLV001_Odin/AvionicsHeartbeat.sch (KiCad schematic (older format))
At the start: 33 parts, among them Q1 DMG2302UK-7, Q2 DMP2123L-7, U1 74HC21, U2 74HC266, U3 74HC08, U4 74HC21, U5 74LVC1G17, U6 LTC6993xS6-1

Commit message: Spec all current parts for Odin
Parts:
- removed C1, C2, C3, C4: 0.1uF, Capacitor_SMD:C_0603_1608Metric_Pad1.05x0.95mm_HandSolder, symbol Device:C
- added C10, C11, C12, C13: 0.1uF, Capacitor_SMD:C_0603_1608Metric_Pad1.05x0.95mm_HandSolder, symbol Device:C
- C6: Digikey 311-1341-1-ND -> (none); MFPN (none) -> CC0603KRX7R8BB104
- C7: footprint (none) -> Capacitor_SMD:C_0603_1608Metric_Pad1.05x0.95mm_HandSolder; MFPN (none) -> CL10B105KA8NNNC
- D2: Digikey 732-4983-1-ND -> (none); MFPN (none) -> 150080GS75000
- D3: Digikey 732-4982-1-ND -> (none); MFPN (none) -> 150080BS75000
- Q1: Digikey DMG2302UK-7DICT-ND -> (none); MFPN (none) -> DMG2302UK-7
- Q2: symbol Device:Q_PMOS_GDS -> Device:Q_PMOS_GSD; Digikey DMP2123LDICT-ND -> (none); MFPN (none) -> DMP2123L-7
- R1, R2, R3, R4, R5, R6, R7, R8: footprint (none) -> Resistor_SMD:R_0603_1608Metric_Pad1.05x0.95mm_HandSolder
- R10: footprint (none) -> Resistor_SMD:R_0603_1608Metric_Pad1.05x0.95mm_HandSolder; MFPN (none) -> RMCF0603FT280K
- R11: footprint (none) -> Resistor_SMD:R_0603_1608Metric_Pad1.05x0.95mm_HandSolder; MFPN (none) -> RMCF0603FT604K
- R12, R14, R15: footprint (none) -> Resistor_SMD:R_0603_1608Metric_Pad1.05x0.95mm_HandSolder; MFPN (none) -> RMCF0603FT47K0
- R16, R17: footprint (none) -> Resistor_SMD:R_0603_1608Metric_Pad1.05x0.95mm_HandSolder; MFPN (none) -> RMCF0603FT1K00
- R9: footprint (none) -> Resistor_SMD:R_0603_1608Metric_Pad1.05x0.95mm_HandSolder; MFPN (none) -> RMCF0603FT1M00
- U1, U4: Digikey 296-31574-1-ND -> (none); MFPN (none) -> CD74HC21M96
- U2: Digikey 296-31804-1-ND -> (none); MFPN (none) -> SN74HC266DR
- U3: Digikey 296-14506-1-ND -> (none); MFPN (none) -> CD74HC08M96
- U3: Digikey 296-14506-1-ND -> CD74HC08M96
- U5: MFPN (none) -> SN74LVC1G17QDBVRQ1
- U6: Digikey LTC6993CS6-1#TRMPBFCT-ND -> (none); MFPN (none) -> LTC6993CS6-1#TRMPBF
Connections:
- net +5V: now also Q2.2 (S), C10.1, C11.1, C12.1, C13.1; no longer Q2.3 (S)
- net GND: now also R15.2, C10.2, C11.2, C12.2, C13.2; no longer R14.2
- net HEARTBEAT: now also Q2.3 (D), R14.2, R15.1; no longer Q2.2 (D), R14.1, R15.2
- net HEARTBEAT_RESTART: now also R14.1; no longer R15.1
